File: module_tests/PD_Filter_Amp/CAD/PD_Filter_Amp.sch (EAGLE design)
At the start: 27 parts, among them IC1 ADA4505-2

Commit message: fixed bug in filter circuit, added test points between each stage
Parts:
- removed C3: CAPACITOR-0.22µF, MABOS_Library:CAPACITOR-0.22µF
- removed C4, C5: CAPACITOR-0.1µF, MABOS_Library:CAPACITOR-0.1µF
- removed R5, R6: RESISTOR-27KOHM, MABOS_Library:RESISTOR-27KOHM
- removed R7: RESISTOR-14KOHM, MABOS_Library:RESISTOR-14KOHM
- added VDD1, VDD2, VDD3, VDD4, VDD5: PAD, Nordic_BLE:PAD
Connections:
- removed net -IN+B: IC1.-IN_B
- removed net N$1: C2.1, C4.1, R4.2, R5.1
- removed net N$2: C3.1, R5.2, R6.1
- removed net N$6: C4.2, C5.1, R7.2
- removed net N$7: C5.2, C6.1, R6.2
- removed net OUT_A: C1.2, GND3.P$1, IC1.OUT_A, R3.2, R4.1
- new net S2_OUT: C1.2, GND3.P$1, IC1.OUT_A, R3.2
- new net S3_IN: R4.1, VDD1.P$1
- new net S3_OUT: C2.1, R4.2, VDD2.P$1
- new net S4_IN: C6.1, VDD3.P$1
- new net S4_OUT: C7.2, R10.2, VDD4.P$1
- new net S5_IN: R11.1, VDD5.P$1
- net +IN_B: no longer C3.2, R7.1
- net -IN_B: now also IC1.-IN_B
- net OUT_B: no longer C7.2, R10.2, R11.1
Other:
- moved on the sheet: C6, C7, C8, R10, R11, R12, R13, R8, R9
